File: Quad Tube VCA.sch (KiCad schematic (older format))
At the start: 212 parts, among them IC1 TL072, IC2 LM358, IC3 TL072, IC4 LM358, IC5 TL072, IC6 LM358, IC7 TL072, IC8 LM358

Commit message: changes footprints for pots/jacks
Parts:
- J_CV_IN1, J_CV_IN2, J_CV_IN3, J_CV_IN4, J_IN2, J_IN3, J_IN4, J_OUT1, J_OUT2, J_OUT3, J_OUT4: footprint Connector_Audio:Jack_3.5mm_QingPu_WQP-PJ398SM_Vertical_CircularHoles -> Eurocad:PJ301M-12
- POT_CV_LEVEL1, POT_CV_LEVEL2, POT_CV_LEVEL3, POT_CV_LEVEL4, POT_FEEDBACK1, POT_FEEDBACK2, POT_FEEDBACK3, POT_FEEDBACK4, POT_GAIN1, POT_GAIN2, POT_GAIN3, POT_GAIN4, POT_IN_DRIVE1, POT_IN_DRIVE2, POT_IN_DRIVE3, POT_IN_DRIVE4: footprint Potentiometer_THT:Potentiometer_Alpha_RD901F-40-00D_Single_Vertical -> Eurocad:Alpha9mmPot
Changed lines of the file:
@@
 F 0 "J_OUT1" H 10272 3889 50  0000 R CNN
 F 1 "PJ301M-12" H 10272 3980 50  0000 R CNN
-F 2 "Connector_Audio:Jack_3.5mm_QingPu_WQP-PJ398SM_Vertical_CircularHoles" H 10272 4071 50  0000 R CNN
+F 2 "Eurocad:PJ301M-12" H 10272 4071 50  0000 R CNN
 F 3 "" H 10750 3950 50  0000 C CNN
 	1    10750 3950
@@
 F 0 "POT_GAIN1" H 3680 5696 50  0000 R CNN
 F 1 "A100k" H 3680 5605 50  0000 R CNN
-F 2 "Potentiometer_THT:Potentiometer_Alpha_RD901F-40-00D_Single_Vertical" H 3750 5650 50  0001 C CNN
+F 2 "Eurocad:Alpha9mmPot" H 3750 5650 50  0001 C CNN
 F 3 "" H 3750 5650 50  0001 C CNN
 	1    3750 5650
@@
 F 0 "J_CV_IN1" H 1873 6284 50  0000 R CNN
 F 1 "PJ301M-12" H 1873 6375 50  0000 R CNN
-F 2 "Connector_Audio:Jack_3.5mm_QingPu_WQP-PJ398SM_Vertical_CircularHoles" H 2350 6300 50  0000 C CNN
+F 2 "Eurocad:PJ301M-12" H 2350 6300 50  0000 C CNN
 F 3 "" H 2350 6300 50  0000 C CNN
 	1    2350 6300
@@
 F 0 "POT_CV_LEVEL1" H 3680 6496 50  0000 R CNN
 F 1 "B100k" H 3680 6405 50  0000 R CNN
-F 2 "Potentiometer_THT:Potentiometer_Alpha_RD901F-40-00D_Single_Vertical" H 3750 6450 50  0001 C CNN
+F 2 "Eurocad:Alpha9mmPot" H 3750 6450 50  0001 C CNN
 F 3 "" H 3750 6450 50  0001 C CNN
 	1    3750 6450
@@
 F 0 "POT_IN_DRIVE1" H 3681 4396 50  0000 R CNN
 F 1 "A100k" H 3681 4305 50  0000 R CNN
-F 2 "Potentiometer_THT:Potentiometer_Alpha_RD901F-40-00D_Single_Vertical" H 3750 4350 50  0001 C CNN
+F 2 "Eurocad:Alpha9mmPot" H 3750 4350 50  0001 C CNN
 F 3 "" H 3750 4350 50  0001 C CNN
 	1    3750 4350
@@
 F 0 "POT_FEEDBACK1" H 3631 3146 50  0000 R CNN
 F 1 "A100k" H 3631 3055 50  0000 R CNN
-F 2 "Potentiometer_THT:Potentiometer_Alpha_RD901F-40-00D_Single_Vertical" H 3700 3100 50  0001 C CNN
+F 2 "Eurocad:Alpha9mmPot" H 3700 3100 50  0001 C CNN
 F 3 "" H 3700 3100 50  0001 C CNN
 	1    3700 3100
@@
 F 0 "POT_FEEDBACK2" H 3631 9046 50  0000 R CNN
 F 1 "A100k" H 3631 8955 50  0000 R CNN
-F 2 "Potentiometer_THT:Potentiometer_Alpha_RD901F-40-00D_Single_Vertical" H 3700 9000 50  0001 C CNN
+F 2 "Eurocad:Alpha9mmPot" H 3700 9000 50  0001 C CNN
 F 3 "" H 3700 9000 50  0001 C CNN
 	1    3700 9000
@@
 F 0 "J_IN2" H 1873 10084 50  0000 R CNN
 F 1 "PJ301M-12" H 1873 10175 50  0000 R CNN
-F 2 "Connector_Audio:Jack_3.5mm_QingPu_WQP-PJ398SM_Vertical_CircularHoles" H 2350 10100 50  0000 C CNN
+F 2 "Eurocad:PJ301M-12" H 2350 10100 50  0000 C CNN
 F 3 "" H 2350 10100 50  0000 C CNN
 	1    2350 10100
@@
 F 0 "POT_IN_DRIVE2" H 3681 10296 50  0000 R CNN
 F 1 "A100k" H 3681 10205 50  0000 R CNN
-F 2 "Potentiometer_THT:Potentiometer_Alpha_RD901F-40-00D_Single_Vertical" H 3750 10250 50  0001 C CNN
+F 2 "Eurocad:Alpha9mmPot" H 3750 10250 50  0001 C CNN
 F 3 "" H 3750 10250 50  0001 C CNN
 	1    3750 10250
@@
 F 0 "POT_CV_LEVEL2" H 3680 12396 50  0000 R CNN
 F 1 "B100k" H 3680 12305 50  0000 R CNN
-F 2 "Potentiometer_THT:Potentiometer_Alpha_RD901F-40-00D_Single_Vertical" H 3750 12350 50  0001 C CNN
+F 2 "Eurocad:Alpha9mmPot" H 3750 12350 50  0001 C CNN
 F 3 "" H 3750 12350 50  0001 C CNN
 	1    3750 12350
@@
 F 0 "J_CV_IN2" H 1873 12184 50  0000 R CNN
 F 1 "PJ301M-12" H 1873 12275 50  0000 R CNN
-F 2 "Connector_Audio:Jack_3.5mm_QingPu_WQP-PJ398SM_Vertical_CircularHoles" H 2350 12200 50  0000 C CNN
+F 2 "Eurocad:PJ301M-12" H 2350 12200 50  0000 C CNN
 F 3 "" H 2350 12200 50  0000 C CNN
 	1    2350 12200
@@
 F 0 "POT_GAIN2" H 3680 11596 50  0000 R CNN
 F 1 "A100k" H 3680 11505 50  0000 R CNN
-F 2 "Potentiometer_THT:Potentiometer_Alpha_RD901F-40-00D_Single_Vertical" H 3750 11550 50  0001 C CNN
+F 2 "Eurocad:Alpha9mmPot" H 3750 11550 50  0001 C CNN
 F 3 "" H 3750 11550 50  0001 C CNN
 	1    3750 11550
@@
 F 0 "J_OUT2" H 10272 9834 50  0000 R CNN
 F 1 "PJ301M-12" H 10272 9925 50  0000 R CNN
-F 2 "Connector_Audio:Jack_3.5mm_QingPu_WQP-PJ398SM_Vertical_CircularHoles" H 10750 9850 50  0000 C CNN
+F 2 "Eurocad:PJ301M-12" H 10750 9850 50  0000 C CNN
 F 3 "" H 10750 9850 50  0000 C CNN
 	1    10750 9850
@@
 F 0 "J_OUT3" H 10272 15834 50  0000 R CNN
 F 1 "PJ301M-12" H 10272 15925 50  0000 R CNN
-F 2 "Connector_Audio:Jack_3.5mm_QingPu_WQP-PJ398SM_Vertical_CircularHoles" H 10750 15850 50  0000 C CNN
+F 2 "Eurocad:PJ301M-12" H 10750 15850 50  0000 C CNN
 F 3 "" H 10750 15850 50  0000 C CNN
 	1    10750 15850
@@
 F 0 "POT_GAIN3" H 3680 17596 50  0000 R CNN
 F 1 "A100k" H 3680 17505 50  0000 R CNN
-F 2 "Potentiometer_THT:Potentiometer_Alpha_RD901F-40-00D_Single_Vertical" H 3750 17550 50  0001 C CNN
+F 2 "Eurocad:Alpha9mmPot" H 3750 17550 50  0001 C CNN
 F 3 "" H 3750 17550 50  0001 C CNN
 	1    3750 17550
@@
 F 0 "J_CV_IN3" H 1873 18184 50  0000 R CNN
 F 1 "PJ301M-12" H 1873 18275 50  0000 R CNN
-F 2 "Connector_Audio:Jack_3.5mm_QingPu_WQP-PJ398SM_Vertical_CircularHoles" H 2350 18200 50  0000 C CNN
+F 2 "Eurocad:PJ301M-12" H 2350 18200 50  0000 C CNN
 F 3 "" H 2350 18200 50  0000 C CNN
 	1    2350 18200
@@
 F 0 "POT_CV_LEVEL3" H 3680 18396 50  0000 R CNN
 F 1 "B100k" H 3680 18305 50  0000 R CNN
-F 2 "Potentiometer_THT:Potentiometer_Alpha_RD901F-40-00D_Single_Vertical" H 3750 18350 50  0001 C CNN
+F 2 "Eurocad:Alpha9mmPot" H 3750 18350 50  0001 C CNN
 F 3 "" H 3750 18350 50  0001 C CNN
 	1    3750 18350
@@
 F 0 "POT_IN_DRIVE3" H 3681 16296 50  0000 R CNN
 F 1 "A100k" H 3681 16205 50  0000 R CNN
-F 2 "Potentiometer_THT:Potentiometer_Alpha_RD901F-40-00D_Single_Vertical" H 3750 16250 50  0001 C CNN
+F 2 "Eurocad:Alpha9mmPot" H 3750 16250 50  0001 C CNN
 F 3 "" H 3750 16250 50  0001 C CNN
 	1    3750 16250
@@
 F 0 "J_IN3" H 1873 16084 50  0000 R CNN
 F 1 "PJ301M-12" H 1873 16175 50  0000 R CNN
-F 2 "Connector_Audio:Jack_3.5mm_QingPu_WQP-PJ398SM_Vertical_CircularHoles" H 2350 16100 50  0000 C CNN
+F 2 "Eurocad:PJ301M-12" H 2350 16100 50  0000 C CNN
 F 3 "" H 2350 16100 50  0000 C CNN
 	1    2350 16100
@@
 F 0 "POT_FEEDBACK3" H 3631 15046 50  0000 R CNN
 F 1 "A100k" H 3631 14955 50  0000 R CNN
-F 2 "Potentiometer_THT:Potentiometer_Alpha_RD901F-40-00D_Single_Vertical" H 3700 15000 50  0001 C CNN
+F 2 "Eurocad:Alpha9mmPot" H 3700 15000 50  0001 C CNN
 F 3 "" H 3700 15000 50  0001 C CNN
 	1    3700 15000
@@
 F 0 "J_OUT4" H 10322 21934 50  0000 R CNN
 F 1 "PJ301M-12" H 10322 22025 50  0000 R CNN
-F 2 "Connector_Audio:Jack_3.5mm_QingPu_WQP-PJ398SM_Vertical_CircularHoles" H 10800 21950 50  0000 C CNN
+F 2 "Eurocad:PJ301M-12" H 10800 21950 50  0000 C CNN
 F 3 "" H 10800 21950 50  0000 C CNN
 	1    10800 21950
@@
 F 0 "POT_GAIN4" H 3730 23696 50  0000 R CNN
 F 1 "A100k" H 3730 23605 50  0000 R CNN
-F 2 "Potentiometer_THT:Potentiometer_Alpha_RD901F-40-00D_Single_Vertical" H 3800 23650 50  0001 C CNN
+F 2 "Eurocad:Alpha9mmPot" H 3800 23650 50  0001 C CNN
 F 3 "" H 3800 23650 50  0001 C CNN
 	1    3800 23650
@@
 F 0 "J_CV_IN4" H 1923 24284 50  0000 R CNN
 F 1 "PJ301M-12" H 1923 24375 50  0000 R CNN
-F 2 "Connector_Audio:Jack_3.5mm_QingPu_WQP-PJ398SM_Vertical_CircularHoles" H 2400 24300 50  0000 C CNN
+F 2 "Eurocad:PJ301M-12" H 2400 24300 50  0000 C CNN
 F 3 "" H 2400 24300 50  0000 C CNN
 	1    2400 24300
@@
 F 0 "POT_CV_LEVEL4" H 3730 24496 50  0000 R CNN
 F 1 "B100k" H 3730 24405 50  0000 R CNN
-F 2 "Potentiometer_THT:Potentiometer_Alpha_RD901F-40-00D_Single_Vertical" H 3800 24450 50  0001 C CNN
+F 2 "Eurocad:Alpha9mmPot" H 3800 24450 50  0001 C CNN
 F 3 "" H 3800 24450 50  0001 C CNN
 	1    3800 24450
@@
 F 0 "POT_IN_DRIVE4" H 3731 22396 50  0000 R CNN
 F 1 "A100k" H 3731 22305 50  0000 R CNN
-F 2 "Potentiometer_THT:Potentiometer_Alpha_RD901F-40-00D_Single_Vertical" H 3800 22350 50  0001 C CNN
+F 2 "Eurocad:Alpha9mmPot" H 3800 22350 50  0001 C CNN
 F 3 "" H 3800 22350 50  0001 C CNN
 	1    3800 22350
@@
 F 0 "J_IN4" H 1923 22184 50  0000 R CNN
 F 1 "PJ301M-12" H 1923 22275 50  0000 R CNN
-F 2 "Connector_Audio:Jack_3.5mm_QingPu_WQP-PJ398SM_Vertical_CircularHoles" H 2400 22200 50  0000 C CNN
+F 2 "Eurocad:PJ301M-12" H 2400 22200 50  0000 C CNN
 F 3 "" H 2400 22200 50  0000 C CNN
 	1    2400 22200
@@
 F 0 "POT_FEEDBACK4" H 3681 21146 50  0000 R CNN
 F 1 "A100k" H 3681 21055 50  0000 R CNN
-F 2 "Potentiometer_THT:Potentiometer_Alpha_RD901F-40-00D_Single_Vertical" H 3750 21100 50  0001 C CNN
+F 2 "Eurocad:Alpha9mmPot" H 3750 21100 50  0001 C CNN
 F 3 "" H 3750 21100 50  0001 C CNN
 	1    3750 21100

Commit message: adds summing mixers to outputs
Parts:
- added C51, C52, C53, C54: 100nf, Capacitor_SMD:C_0603_1608Metric, symbol Device:C_Small
- added IC10, IC9: TL072, Package_SO:SOIC-8_3.9x4.9mm_P1.27mm, symbol Amplifier_Operational:TL072
- added R84, R85, R86, R87, R88, R89, R90, R91: 100k, Resistor_SMD:R_0603_1608Metric, symbol Device:R_Small_US
Connections:
- net +12V: now also C51.1, C53.1, IC10.8 (V+), IC9.8 (V+)
- net -12V: now also C52.2, C54.2, IC10.4 (V-), IC9.4 (V-)
- net GND: now also C51.2, C52.1, C53.2, C54.1, IC10.3 (+), IC10.5 (+), IC9.3 (+), IC9.5 (+)
- net at C4.2, IC1.7: now also R1.1, R3.2, R81.2; no longer R8.1
- net at J_OUT1.3, R8.2: no longer R1.1, R3.2
- net at J_OUT1.2: now also R85.2; no longer R81.1
- net at C15.2, IC3.2 (-), R24.2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: no longer R81.2
- net at R21.1, R23.2: now also C16.2, IC3.7, R82.2; no longer J_OUT2.3, R28.2
- net at R82.1: now also IC9.6 (-), R85.1, R89.2; no longer J_OUT2.2
- net at C27.2, IC5.2 (-), R44.2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: no longer R82.2
- net at R41.1, R43.2: now also C28.2, IC5.7, R83.2; no longer J_OUT3.3, R48.2
- net at R83.1: now also IC10.2 (-), R86.1, R90.2; no longer J_OUT3.2
- net at C39.2, IC7.2 (-), R64.2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: no longer R83.2
- net at R61.1, R63.2: now also C40.2, IC7.7, R84.2; no longer J_OUT4.3, R68.2
- new net: IC9.1, R8.1, R88.1
- new net: IC9.2 (-), R81.1, R88.2
- new net: IC9.7, R28.1, R89.1
- new net: J_OUT2.2, R86.2
- new net: J_OUT2.3, R28.2
- new net: IC10.1, R48.1, R90.1
- new net: IC10.6 (-), R84.1, R87.1, R91.2
- new net: IC10.7, R68.1, R91.1
- new net: J_OUT3.2, R87.2
- new net: J_OUT3.3, R48.2
- new net: J_OUT4.3, R68.2
- no-connect marks 0 -> 1
Other:
- moved on the sheet: C10, C11, C12, C13, C2, C22, C23, C24, C25, C3, C34, C35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

Commit message: updates footprints in schematic
Parts:
- C19, C2, C3, C31, C43, C7: footprint Capacitor_THT:CP_Radial_D7.5mm_P2.50mm -> Capacitor_THT:CP_Radial_D5.0mm_P2.50mm
- SW_DIST1, SW_DIST2, SW_DIST3, SW_DIST4: footprint Button_Switch_THT:SW_Lever_1P2T_NKK_GW12LxH -> 100SP1T1B4M2QE:SW_100SP1T1B4M2QE
Changed lines of the file:
@@
 F 0 "C2" H 13850 2100 50  0000 L CNN
 F 1 "10uf" H 13700 2250 50  0000 L CNN
-F 2 "Capacitor_THT:CP_Radial_D7.5mm_P2.50mm" H 13750 2100 50  0001 C CNN
+F 2 "Capacitor_THT:CP_Radial_D5.0mm_P2.50mm" H 13750 2100 50  0001 C CNN
 F 3 "" H 13750 2100 50  0001 C CNN
 	1    13750 2100
@@
 F 0 "C3" H 13850 2300 50  0000 L CNN
 F 1 "10uf" H 13700 2150 50  0000 L CNN
-F 2 "Capacitor_THT:CP_Radial_D7.5mm_P2.50mm" H 13750 2300 50  0001 C CNN
+F 2 "Capacitor_THT:CP_Radial_D5.0mm_P2.50mm" H 13750 2300 50  0001 C CNN
 F 3 "" H 13750 2300 50  0001 C CNN
 	1    13750 2300
@@
 F 0 "SW_DIST1" V 6696 4048 50  0000 L CNN
 F 1 "SW_SPDT" V 6605 4048 50  0000 L CNN
-F 2 "Button_Switch_THT:SW_Lever_1P2T_NKK_GW12LxH" H 6650 3900 50  0001 C CNN
+F 2 "100SP1T1B4M2QE:SW_100SP1T1B4M2QE" H 6650 3900 50  0001 C CNN
 F 3 "" H 6650 3900 50  0001 C CNN
 	1    6650 3900
@@
 F 0 "C7" H 8163 5004 50  0000 R CNN
 F 1 "47uf" H 8163 5095 50  0000 R CNN
-F 2 "Capacitor_THT:CP_Radial_D7.5mm_P2.50mm" H 8250 5050 50  0001 C CNN
+F 2 "Capacitor_THT:CP_Radial_D5.0mm_P2.50mm" H 8250 5050 50  0001 C CNN
 F 3 "" H 8250 5050 50  0001 C CNN
 	1    8250 5050
@@
 F 0 "C19" H 8163 10904 50  0000 R CNN
 F 1 "47uf" H 8163 10995 50  0000 R CNN
-F 2 "Capacitor_THT:CP_Radial_D7.5mm_P2.50mm" H 8250 10950 50  0001 C CNN
+F 2 "Capacitor_THT:CP_Radial_D5.0mm_P2.50mm" H 8250 10950 50  0001 C CNN
 F 3 "" H 8250 10950 50  0001 C CNN
 	1    8250 10950
@@
 F 0 "SW_DIST2" V 6696 9948 50  0000 L CNN
 F 1 "SW_SPDT" V 6605 9948 50  0000 L CNN
-F 2 "Button_Switch_THT:SW_Lever_1P2T_NKK_GW12LxH" H 6650 9800 50  0001 C CNN
+F 2 "100SP1T1B4M2QE:SW_100SP1T1B4M2QE" H 6650 9800 50  0001 C CNN
 F 3 "" H 6650 9800 50  0001 C CNN
 	1    6650 9800
@@
 F 0 "SW_DIST3" V 6696 15948 50  0000 L CNN
 F 1 "SW_SPDT" V 6605 15948 50  0000 L CNN
-F 2 "Button_Switch_THT:SW_Lever_1P2T_NKK_GW12LxH" H 6650 15800 50  0001 C CNN
+F 2 "100SP1T1B4M2QE:SW_100SP1T1B4M2QE" H 6650 15800 50  0001 C CNN
 F 3 "" H 6650 15800 50  0001 C CNN
 	1    6650 15800
@@
 F 0 "C31" H 8163 16904 50  0000 R CNN
 F 1 "47uf" H 8163 16995 50  0000 R CNN
-F 2 "Capacitor_THT:CP_Radial_D7.5mm_P2.50mm" H 8250 16950 50  0001 C CNN
+F 2 "Capacitor_THT:CP_Radial_D5.0mm_P2.50mm" H 8250 16950 50  0001 C CNN
 F 3 "" H 8250 16950 50  0001 C CNN
 	1    8250 16950
@@
 F 0 "SW_DIST4" V 6746 22048 50  0000 L CNN
 F 1 "SW_SPDT" V 6655 22048 50  0000 L CNN
-F 2 "Button_Switch_THT:SW_Lever_1P2T_NKK_GW12LxH" H 6700 21900 50  0001 C CNN
+F 2 "100SP1T1B4M2QE:SW_100SP1T1B4M2QE" H 6700 21900 50  0001 C CNN
 F 3 "" H 6700 21900 50  0001 C CNN
 	1    6700 21900
@@
 F 0 "C43" H 8213 23004 50  0000 R CNN
 F 1 "47uf" H 8213 23095 50  0000 R CNN
-F 2 "Capacitor_THT:CP_Radial_D7.5mm_P2.50mm" H 8300 23050 50  0001 C CNN
+F 2 "Capacitor_THT:CP_Radial_D5.0mm_P2.50mm" H 8300 23050 50  0001 C CNN
 F 3 "" H 8300 23050 50  0001 C CNN
 	1    8300 23050
